File: hardware/led_controller/led_controller.kicad_pcb (KiCad board)
At the start: 2 copper layers, 99.9 x 79.3 mm, 65 parts, among them J1 LED3, J10 POWER, J11 POWER, J12 I2C, J2 POWER, J3 LIGHT_SENSOR, J4 LED_1, J5 USB, J6 OLED, J7 FLASH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

Commit message: added last pcb verison
Parts:
- C1, C3: footprint Capacitor_THT:CP_Radial_D5.0mm_P2.50mm -> Capacitor_THT:CP_Radial_D7.5mm_P2.50mm
- moved C7 1.84 mm to (154.3, 77.7), turned to 180 degrees
- moved C3 1.04 mm to (155.6, 69.1)
Connections:
- C1 pad 1: EN -> IN-
- C6 pad 1: EN -> IN-
- C7 pad 1: EN -> IN-
- C8 pad 1: EN -> IN-
- D4 pad 2: EN -> IN-
- J1 pad 1: EN -> IN-
- J10 pad 2: EN -> IN-
- J11 pad 2: EN -> IN-
- J4 pad 1: EN -> IN-
- J8 pad 2: EN -> IN-
- J9 pad 2: EN -> IN-
- R20 pad 1: EN -> IN-
- R21 pad 2: EN -> IN-
- R7 pad 1: EN -> GND
- U8 pad 7: EN -> IN-
Routing:
- net EN: track 309.5 -> 0.00 mm, vias 4 -> 0
- net IN-: track 0.00 -> 301.5 mm, vias 0 -> 3
- net Net-(U1-~{EN}): track 28.9 -> 29.6 mm, vias 2 -> 3
